File: Hardware/OpenLog.sch (EAGLE design)
At the start: 30 parts, among them J2 SMD, J3 PTH, J4 SMD, J5 ISP, Q1 16MHZ, U2 ATMEGA328P, U3 microSD Socket

Commit message: More examples. Finishing up v1.0.
Other:
- note added: "Closed = 0x29"
- note added: "Open (default) = 0x2A"
- note removed: "Closed = 0x43"
- note removed: "Open (default) = 0x42"
Changed lines of the file:
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@@
 <wire x1="81.28" y1="185.42" x2="81.28" y2="35.56" width="0.2032" layer="97" style="shortdash"/>
 <text x="180.34" y="53.34" size="1.778" layer="97">7-Bit I2C Address Jumper</text>
-<text x="182.88" y="48.26" size="1.778" layer="97">Closed = 0x43</text>
-<text x="182.88" y="50.8" size="1.778" layer="97">Open (default) = 0x42</text>
+<text x="182.88" y="48.26" size="1.778" layer="97">Closed = 0x29</text>
+<text x="182.88" y="50.8" size="1.778" layer="97">Open (default) = 0x2A</text>
 </plain>
 <instances>
